File: Project/pandemonium BLE.kicad_sch (KiCad schematic)
At the start: 123 parts, among them J5 SWD_TC2030, SW1 RotaryEncoder_Switch, SW2 RotaryEncoder_Switch, SW44 RST, U1 nRF52840, Y1 32.768 KHz, Y2 32 MHz

Commit message: EC version finished
Parts:
- SW44: footprint PCM_marbastlib-various:SW_SPST_SKQG_WithStem -> Button_Switch_SMD:SW_Push_SPST_NO_Alps_SKRK
Connections:
- net r0 is gone; now on net COL7: U1.A12 (AIN0/P0.02)
- net r4 is gone; now on net COL3: U1.J1 (AIN2/P0.04)
- net COL0: now also U1.AD16 (P0.20)
- net COL1: now also U1.L24 (NFC1/P0.09)
- net COL2: now also U1.L1 (P0.06)
- net COL4: now also U1.A8 (AIN7/P0.31)
- net COL5: now also U1.A10 (AIN5/P0.29)
- net COL6: now also U1.A20 (P1.10)
- net COL8: now also U1.A14 (P1.15)
- net COL9: now also U1.A16 (P1.13)
- net ROTARY_A: now also U1.N1 (P0.08)
- net ROTARY_B: now also U1.R1 (TRACEDATA3/P1.09)
- net ROW0: now also U1.AD8 (P0.13)
- net ROW1: now also U1.AD10 (P0.15)
- net ROW2: now also U1.AD18 (P0.22)
- net ROW3: now also U1.U1 (TRACEDATA1/P0.12)
- net SDA: now reaches U1.AD20 (P0.24)
- net SCL: now reaches U1.AD22 (TRACEDATA0/P1.00)
Other:
- moved on the sheet: AE1, C1, C2, C3, C4, C5, C6, C7, J5, L1, LED1, R3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

Commit message: small work on pandi EC and BLE
Parts:
- removed LED1: blue, LED_SMD:LED_0402_1005Metric, symbol Device:LED_Small
- removed R3: 1 kOhm, Resistor_SMD:R_0402_1005Metric, symbol Device:R_Small
- added U6: nRF52840_holyiot_18010, PCM_marbastlib-various:nRF52840_holyiot_18010, symbol PCM_marbastlib-various:nRF52840_holyiot_18010
Connections:
- net GND: now also U6.1 (GND), U6.25 (GND), U6.37 (GND)
- net RESET: now also U6.21 (P0.18-RESET)
- net LED: no longer names the net of U1.W24 (P1.02)
- new net D+: U6.24 (D+)
- new net D-: U6.23 (D-)
- new net SWC: U6.31 (SWDCLK)
- new net SWD: U6.32 (SWDIO)
- new net VDD_NRF: U6.14 (VDD_nRF)

Commit message: switching to holyiot for BLE
Parts:
- removed AE1: 2.4 GHz ANT, RF_Antenna:Texas_SWRA117D_2.4GHz_Left, symbol Device:Antenna_Dipole
- removed C1, C2, C6, C7: 12 pF, Capacitor_SMD:C_0402_1005Metric, symbol Device:C_Small
- removed C12: 100 pF, Capacitor_SMD:C_0402_1005Metric, symbol Device:C_Small
- removed C13, C16, C17, C18: 100 nF, Capacitor_SMD:C_0402_1005Metric, symbol Device:C_Small
- removed C14, C8: 1 uF, Capacitor_SMD:C_0402_1005Metric, symbol Device:C_Small
- removed C15, C19, C20: 4.7 uF, Capacitor_SMD:C_0402_1005Metric, symbol Device:C_Small
- removed C4: 0.5 pF, Capacitor_SMD:C_0402_1005Metric, symbol Device:C_Small
- removed C5: 0.8 pF, Capacitor_SMD:C_0402_1005Metric, symbol Device:C_Small
- removed J5: SWD_TC2030, PCM_marbastlib-various:CON_TC2030_outlined, symbol marbastlib-various:JTAG_TC2030
- removed L1: 4.7 nH, Inductor_SMD:L_0402_1005Metric, symbol Device:L_Small
- removed L2, L4: 10 uH, Inductor_SMD:L_0603_1608Metric, symbol Device:L_Small
- removed L3: 15 nH, Inductor_SMD:L_0402_1005Metric, symbol Device:L_Small
- removed SW44: RST, Button_Switch_SMD:SW_Push_SPST_NO_Alps_SKRK, symbol Switch:SW_SPST
- removed U1: nRF52840, Package_DFN_QFN:Nordic_AQFN-73-1EP_7x7mm_P0.5mm, symbol MCU_Nordic:nRF52840
- removed Y1: 32.768 KHz, Crystal:Crystal_SMD_2012-2Pin_2.0x1.2mm, symbol Device:Crystal_Small
- removed Y2: 32 MHz, Crystal:Crystal_SMD_2016-4Pin_2.0x1.6mm, symbol Device:Crystal_GND24_Small
- added C2, C4: 10 uF, symbol Device:C_Polarized_Small
- added D2: Schottky, symbol Device:D_Schottky
- added J3: Battery, Connector_JST:JST_PH_S2B-PH-K_1x02_P2.00mm_Horizontal, symbol Connector_Generic_MountingPin:Conn_01x02_MountingPin
- added J7: TC2030_SWD, PCM_marbastlib-various:CON_TC2030_outlined, symbol PCM_marbastlib-various:TC2030_SWD
- added LED1: orange, LED_SMD:LED_0402_1005Metric, symbol Device:LED_Small
- added Q1: AO3401A, Package_TO_SOT_SMD:SOT-23, symbol Transistor_FET:AO3401A
- added R21: 806 kOhm, Resistor_SMD:R_0402_1005Metric, symbol Device:R_Small
- added R22: 2 MOhm, Resistor_SMD:R_0402_1005Metric, symbol Device:R_Small
- added R6, R7: 1.5 kOhm, Resistor_SMD:R_0402_1005Metric, symbol Device:R_Small
- added R9: 5 kOhm, Resistor_SMD:R_0402_1005Metric, symbol Device:R_Small
- added SW2: PWR, PCM_marbastlib-various:SW_MSK12C02-HB, symbol Switch:SW_Push_SPDT
- added SW3: RESET, PCM_marbastlib-various:SW_SPST_SKQG_WithStem, symbol Switch:SW_Push_45deg
- added U2: TP4056, Package_SO:SOP-8-1EP_4.57x4.57mm_P1.27mm_EP4.57x4.45mm, symbol PCM_marbastlib-various:TP4056
- added U6: XC6206PxxxMR, Package_TO_SOT_SMD:SOT-23, symbol Regulator_Linear:XC6206PxxxMR
- C10: value 4.7 uF -> 1 uF; LCSC C23733 -> (none)
- C11: value 820 pF -> 100 nF; LCSC C161159 -> (none); Notes NP0, 5% -> X7R, 10%
- C3: value NC -> 4.7 uF; LCSC C77179 -> (none); Notes (none) -> X7R, 10%; now in the parts list
- C9: value 47 nF -> 1 uF; LCSC C26403 -> (none)
- S1, S5: value MX_stab -> ISO
- S2, S3, S4: value MX_stab -> 3
- S6, S7: value MX_stab -> 225
- S8: value MX_stab -> 6
- S9: value MX_stab -> 7
Connections:
- net D+ is gone; now on net USB-Do+: U6.24 (D+)
- net D- is gone; now on net USB-Do-: U6.23 (D-)
- net DEC4_6 is gone; now on net +VSW: C9.1
- net SWD is gone; now on net SWDIO: U6.32 (SWDIO)
- net +5V: now also C3.1, U6.22 (VBUS), C2.1, D2.2 (A), LED1.2 (A), Q1.1 (G), R7.1, U2.4 (VCC), U2.8 (CE)
- net +VSW: now also D2.1 (K), Q1.2 (S), R21.1, U6.3 (VI); no longer C10.1
- net COL0: now also D1.2 (A), D3.2 (A), D5.2 (A), D7.2 (A); no longer MX1.1, MX3.1, MX5.1, MX7.1
- net COL1: now also D10.2 (A), D12.2 (A), D8.2 (A); no longer MX10.1, MX12.1, MX8.1
- net COL2: now also D14.2 (A), D15.2 (A), D17.2 (A), D19.2 (A); no longer MX14.1, MX15.1, MX17.1, MX19.1, MX36.1, SW1.S2
- net COL3: now also D21.2 (A), D22.2 (A), D28.2 (A), D34.2 (A); no longer MX21.1, MX22.1, MX24.1, MX26.1, MX35.1, MX37.1, MX38.1
- net COL4: now also D23.2 (A), D29.2 (A), D35.2 (A); no longer MX29.1, MX31.1, MX33.1, MX34.1, MX39.1, SW2.S2
- net COL5: now also D2.2 (A), D24.2 (A), D4.2 (A), D6.2 (A); no longer MX2.1, MX28.1, MX4.1, MX42.1, MX43.1, MX6.1
- net COL6: now also D11.2 (A), D13.2 (A), D40.2 (A), D9.2 (A); no longer MX11.1, MX13.1, MX9.1
- net COL7: now also D16.2 (A), D18.2 (A), D20.2 (A); no longer MX16.1, MX18.1, MX20.1, MX44.1
- net COL8: now also D25.2 (A), D27.2 (A), D31.2 (A), D37.2 (A); no longer MX23.1, MX25.1, MX40.1
- net COL9: now also D26.2 (A), D30.2 (A), D32.2 (A); no longer MX27.1, MX30.1, MX32.1, MX41.1
- net GND: now also C3.2, C2.2, C4.2, J3.2 (Pin_2), J3.MP (MountPin), J7.5 (GND), R22.2, R7.2, R9.2, SW3.2, U2.1 (TEMP), U2.3 (GND), U6.1 (GND); no longer C3.1
- net ROW0: now also MX1.1, MX15.1, MX16.1, MX2.1, MX22.1, MX23.1, MX29.1, MX30.1, MX8.1, MX9.1; no longer D1.1 (K), D15.1 (K), D16.1 (K), D2.1 (K), D22.1 (K), D23.1 (K), D25.1 (K), D26.1 (K), D8.1 (K), D9.1 (K)
- net ROW1: now also MX10.1, MX11.1, MX17.1, MX18.1, MX24.1, MX25.1, MX3.1, MX31.1, MX32.1, MX4.1; no longer D10.1 (K), D11.1 (K), D17.1 (K), D18.1 (K), D28.1 (K), D29.1 (K), D3.1 (K), D31.1 (K), D32.1 (K), D4.1 (K)
- net ROW2: now also MX12.1, MX13.1, MX19.1, MX20.1, MX26.1, MX27.1, MX33.1, MX40.1, MX41.1, MX5.1, MX6.1; no longer D12.1 (K), D13.1 (K), D19.1 (K), D20.1 (K), D34.1 (K), D35.1 (K), D37.1 (K), D5.1 (K), D6.1 (K)
- net ROW3: now also MX14.1, MX21.1, MX28.1, MX34.1, MX35.1, MX36.1, MX37.1, MX38.1, MX39.1, MX42.1, MX43.1, MX44.1, MX7.1, SW1.S2, SW2.S2; no longer D14.1 (K), D21.1 (K), D24.1 (K), D27.1 (K), D30.1 (K), D40.1 (K), D7.1 (K)
- net SCL: now also U6.13 (P0.05-A)
- net SDA: now also U6.15 (P0.07)
- net SWDCLK: now also J7.4 (SWCLK)
- net SWDIO: now also J7.2 (SWDIO)
- net VDD_NRF: no longer U6.14 (VDD_nRF)
- net row1: now also D14.1 (K); no longer D14.2 (A)
- net row2: now also D24.1 (K); no longer D24.2 (A)
- net at MX13.2: now also D13.1 (K); no longer D13.2 (A)
- net at MX17.2: now also D17.1 (K); no longer D17.2 (A)
- net at MX4.2: now also D4.1 (K); no longer D4.2 (A)
- net at MX23.2: now also D25.1 (K); no longer D25.2 (A)
- net at MX21.2, MX35.2, MX37.2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: now also D21.1 (K); no longer D21.2 (A)
- net at MX28.2, MX42.2, MX43.2: now also D40.1 (K); no longer D40.2 (A)
- net at MX18.2: now also D18.1 (K); no longer D18.2 (A)
- net at MX3.2: now also D3.1 (K); no longer D3.2 (A)
- net at MX24.2: now also D28.1 (K); no longer D28.2 (A)
- net at MX30.2: now also D26.1 (K); no longer D26.2 (A)
- net at MX27.2, MX41.2: now also D37.1 (K); no longer D37.2 (A)
- net at MX44.2: now also D27.1 (K); no longer D27.2 (A)
- net at MX16.2: now also D16.1 (K); no longer D16.2 (A)
- net at MX19.2: now also D19.1 (K); no longer D19.2 (A)
- net at MX10.2: now also D10.1 (K); no longer D10.2 (A)
- net at MX7.2: now also D7.1 (K); no longer D7.2 (A)
- net at MX1.2: now also D1.1 (K); no longer D1.2 (A)
- net at MX5.2: now also D5.1 (K); no longer D5.2 (A)
- net at MX32.2: now also D32.1 (K); no longer D32.2 (A)
- net at MX22.2: now also D22.1 (K); no longer D22.2 (A)
- net at MX20.2: now also D20.1 (K); no longer D20.2 (A)
- net at MX15.2: now also D15.1 (K); no longer D15.2 (A)
- net at MX25.2: now also D31.1 (K); no longer D31.2 (A)
- net at MX9.2: now also D9.1 (K); no longer D9.2 (A)
- net at MX2.2: now also D2.1 (K); no longer D2.2 (A)
- net at MX6.2: now also D6.1 (K); no longer D6.2 (A)
- net at MX29.2: now also D23.1 (K); no longer D23.2 (A)
- net at MX31.2: now also D29.1 (K); no longer D29.2 (A)
- net at MX8.2: now also D8.1 (K); no longer D8.2 (A)
- net VSENSE: now reaches U6.11 (P0.31-LF-A)
- net VSENSE: now also R21.2, R22.1
- net at MX26.2: now also D34.1 (K); no longer D34.2 (A)
- net at MX12.2: now also D12.1 (K); no longer D12.2 (A)
- net at MX33.2: now also D35.1 (K); no longer D35.2 (A)
- net at MX40.2: now also D30.1 (K); no longer D30.2 (A)
- net at MX11.2: now also D11.1 (K); no longer D11.2 (A)
- net DEC5 renamed +3.3V
- net +3.3V: now also C10.1, J7.1 (VCC), U6.2 (VO)
- net RESET renamed RST
- net RST: now also J7.3 (~{RST}), SW3.1
- net SWC renamed SWCLK
- new net: J3.1 (Pin_1), SW2.2 (B)
- new net: R9.1, U2.2 (PROG)
- new net: R6.2, U2.7 (CHRG)
- new net: LED1.1 (K), R6.1
- new net +3V3: U6.14 (VDD_nRF)
- new net +BATT: C4.1, Q1.3 (D), SW2.1 (A), U2.5 (BAT)
- no-connect marks 27 -> 3
Other:
- note added: "Battery Management (Simple)"
- note added: "MCU Holyiot"
- note added: "PROG: 5 kOhm -> 250 mA charging current TEMP: Pulled to GND -> no OTP"
- note added: "Voltage sensing (simple) - Holyiot only!"
- moved on the sheet: D1, D10, D11, D12, D13, D14, D15, D16, D17, D18, D19, D2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

Commit message: BLE progress
Parts:
- removed C10, C9: 1 uF, Capacitor_SMD:C_0402_1005Metric, symbol Device:C_Small
- removed C11: 100 nF, Capacitor_SMD:C_0402_1005Metric, symbol Device:C_Small
- removed C2, C4: 10 uF, symbol Device:C_Polarized_Small
- removed C3: 4.7 uF, Capacitor_SMD:C_0402_1005Metric, symbol Device:C_Small
- removed D2: Schottky, symbol Device:D_Schottky
- removed LED1: orange, LED_SMD:LED_0402_1005Metric, symbol Device:LED_Small
- removed R21: 806 kOhm, Resistor_SMD:R_0402_1005Metric, symbol Device:R_Small
- removed R22: 2 MOhm, Resistor_SMD:R_0402_1005Metric, symbol Device:R_Small
- removed R7: 1.5 kOhm, Resistor_SMD:R_0402_1005Metric, symbol Device:R_Small
- removed R9: 5 kOhm, Resistor_SMD:R_0402_1005Metric, symbol Device:R_Small
- removed SW2: PWR, PCM_marbastlib-various:SW_MSK12C02-HB, symbol Switch:SW_Push_SPDT
- removed SW3: RESET, PCM_marbastlib-various:SW_SPST_SKQG_WithStem, symbol Switch:SW_Push_45deg
- removed U2: TP4056, Package_SO:SOP-8-1EP_4.57x4.57mm_P1.27mm_EP4.57x4.45mm, symbol PCM_marbastlib-various:TP4056
- removed U6: XC6206PxxxMR, Package_TO_SOT_SMD:SOT-23, symbol Regulator_Linear:XC6206PxxxMR
- removed U6: nRF52840_holyiot_18010, PCM_marbastlib-various:nRF52840_holyiot_18010, symbol PCM_marbastlib-various:nRF52840_holyiot_18010
- added D33: BLUE, LED_SMD:LED_1206_3216Metric_ReverseMount_Hole1.8x2.4mm, symbol Device:LED_Small
- added D38: 1N5819, Diode_SMD:D_SOD-123, symbol Device:D_Small
- added D39: RED, LED_SMD:LED_1206_3216Metric_ReverseMount_Hole1.8x2.4mm, symbol Device:LED_Small
- added F1: 750 mA, Fuse:Fuse_0603_1608Metric, symbol Device:Fuse_Small
- added J1: HRO_TYPE-C-31-M-14, PCM_marbastlib-various:USB_C_Receptacle_HRO_TYPE-C-31-M-12, symbol Connector:USB_C_Receptacle_USB2.0
- added L5: BLM15PX121SN1D, Inductor_SMD:L_0402_1005Metric, symbol Device:L_Small
- added R1, R3: 1K, Resistor_SMD:R_0402_1005Metric, symbol Device:R_Small
- added R2: 810K, Resistor_SMD:R_0402_1005Metric, symbol Device:R_Small
- added R4, R5: 5.1k, Resistor_SMD:R_0402_1005Metric, symbol Device:R_Small
- added R4: 3.3K, Resistor_SMD:R_0402_1005Metric, symbol Device:R_Small
- added R5: 2M, Resistor_SMD:R_0402_1005Metric, symbol Device:R_Small
- added SW3: SW_DPDT, PCM_marbastlib-various:SW_MSK12C02-HB, symbol TK44:MSK12C02
- added SWT1: SW_Push, Button_Switch_SMD:SW_Push_SPST_NO_Alps_SKRK, symbol Switch:SW_Push
- added U2: HOLYIOT-18010, PCM_marbastlib-various:nRF52840_holyiot_18010, symbol TK44:HOLYIOT-18010
- added U3: MCP73831, Package_TO_SOT_SMD:SOT-23-5, symbol Battery_Management:MCP73832-2-OT
- added U4: USBLC6-2P6, Package_TO_SOT_SMD:SOT-666, symbol Power_Protection:USBLC6-2P6
- added U7: XC6220-3.3V, Package_TO_SOT_SMD:SOT-23-5, symbol TK44:AP2112K-3.3V
- Q1: value AO3401A -> AO3407
- R6: value 1.5 kOhm -> 100K
Connections:
- net +5V is gone; now on net VBUS: Q1.1 (G)
- net +BATT is gone; now on net VBAT: Q1.3 (D)
- net COL0: now also U2.20 (P0.19)
- net COL1: now also U2.19 (P0.21)
- net COL2: now also U2.18 (P0.23)
- net COL3: now also U2.17 (P0.12)
- net COL4: now also U2.16 (P1.09)
- net COL5: now also U2.15 (P0.07)
- net COL6: now also U2.13 (P0.05/AIN3)
- net COL7: now also U2.12 (P0.04/AIN2)
- net COL8: now also U2.6 (P0.03/AIN1)
- net COL9: now also U2.5 (P1.15)
- net GND: now also R6.2, J1.A1 (GND), J1.A12 (GND), J1.B1 (GND), J1.B12 (GND), J1.S1 (SHIELD), R1.2, R4.2, R4.2, R5.2, R5.2, SWT1.2, U2.1 (GND), U2.25 (GND), U2.37 (GND), U3.2 (VSS), U4.2 (GND), U7.2 (GND)
- net ROTARY_A: now also U2.9 (P0.29/AIN5)
- net ROTARY_B: now also U2.11 (P0.31/AIN7)
- net ROW0: now also U2.27 (P1.00)
- net ROW1: now also U2.3 (P1.10)
- net ROW2: now also U2.8 (P0.28/AIN4)
- net ROW3: now also U2.10 (P0.30/AIN6)
- net VBAT: now reaches J3.1 (Pin_1)
- net VBAT: now also R2.1, SW3.2, U3.3 (VBAT)
- net VBUS: now reaches R6.1
- net VBUS: now also D38.2 (A), D39.2 (A), F1.2, J1.A4 (VBUS), J1.A9 (VBUS), J1.B4 (VBUS), J1.B9 (VBUS), L5.1, U2.22 (VBUS), U3.4 (VDD), U4.5 (VBUS)
- net +3.3V renamed nRF_VDD
- net nRF_VDD: now also U2.14 (VDD), U7.5 (VOUT)
- net +VSW: no longer names the net of Q1.2 (S)
- net +VSW: now also D38.1 (K), U7.1 (VIN), U7.3 (EN)
- net RST renamed RESET
- net RESET: now also SWT1.1, U2.21 (P0.18/RESET)
- net SWDCLK renamed SWC
- net SWC: now also U2.31 (SWDCLK)
- net SWDIO renamed SWD
- net SWD: now also U2.32 (SWDIO)
- new net: D33.1 (K), R1.1
- new net: D39.1 (K), R3.1
- new net: R3.2, U3.1 (STAT)
- new net: F1.1, L5.2
- new net: R4.1, U3.5 (PROG)
- new net BLUE_LED: D33.2 (A), U2.26 (P0.22)
- new net BT_PIN: R2.2, R5.1, U2.7 (P0.02/AIN0)
- new net CC1: J1.A5 (CC1), R4.1
- new net CC2: J1.B5 (CC2), R5.1
- new net DATA ESD+: J1.A6 (D+), J1.B6 (D+), U4.6 (I/O1)
- new net DATA ESD-: J1.A7 (D-), J1.B7 (D-), U4.4 (I/O2)
- new net DATA+: U2.24 (USB_D+), U4.1 (I/O1)
- new net DATA-: U2.23 (USB_D-), U4.3 (I/O2)
- new net P0.09: U2.35 (P0.09/NFC1)
- new net P0.10: U2.36 (P0.10/NFC2)
- new net P1.01: U2.29 (P1.01)
- new net P1.02: U2.30 (P1.02)
- new net P1.03: U2.28 (P1.03)
- new net P1.04: U2.33 (P1.04)
- new net P1.06: U2.34 (P1.06)
- new net P1.11: U2.2 (P1.11)
- new net P1.13: U2.4 (P1.13)
- no-connect marks 3 -> 4
Other:
- removed sheet Battey Management
- removed sheet USB
- note added: "Battery Сonnector"
- note added: "Charger and blue LED"
- note added: "MATRIX"
- note added: "PINOUT"
- note added: "Power"
- note added: "Reset Button"
- note added: "SWD Сonnector"
- note added: "USB and ESD"
- note removed: "Battery Management (Simple)"
- note removed: "PROG: 5 kOhm -> 250 mA charging current TEMP: Pulled to GND -> no OTP"
- note removed: "Voltage sensing (simple) - Holyiot only!"
- moved on the sheet: D1, D10, D11, D12, D13, D14, D15, D16, D17, D18, D19, D2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

Commit message: EC plates created
Parts:
- removed SW3: SW_DPDT, PCM_marbastlib-various:SW_MSK12C02-HB, symbol TK44:MSK12C02
- added U1, U5, U6: 74LVC1G08, Package_TO_SOT_SMD:SOT-353_SC-70-5, symbol 74xGxx:74LVC1G08
Connections:
- net COL0: now also U1.1, U6.1
- net COL8: now also U6.2
- net COL9: now also U1.2
- net GND: now also U1.3 (GND), U5.3 (GND), U6.3 (GND)
- net nRF_VDD: now also U1.5 (VCC), U5.5 (VCC), U6.5 (VCC)
- net P0.10 renamed WAKESLEEP
- net WAKESLEEP: now also U5.4
- new net: U1.4, U5.1
- new net: U5.2, U6.4
- no-connect marks 4 -> 3
Other:
- note added: "hardware/software wakeup"
- moved on the sheet: F1, J1, J3, J7, L5, R4, R5, SWT1, U4

Commit message: backup
Parts:
- added U8: XC6206PxxxMR, Package_TO_SOT_SMD:SOT-23-3, symbol Regulator_Linear:XC6206PxxxMR
Connections:
- net row1 renamed r1
- net row2 renamed r2
Other:
- note added: "CHANGE LDO, ADD SIMPLE PUSH BUTTON FOR solution, needs GPIO EVQP4HB3B"
Changed lines of the file:
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@@
     (fill (type none))
+  )
+  (text "CHANGE LDO,\n\nADD SIMPLE PUSH BUTTON FOR solution, needs GPIO\n\nEVQP4HB3B"
+    (at 138.43 207.645 0)
+    (effects (font (size 4 4)) (justify left bottom))
   )
   (text "hardware/software wakeup" (at 287.655 66.675 0)
@@
     )
   )
-  (global_label "row1" (shape input) (at 152.4 84.455 0) (fields_autoplaced)
+  (global_label "r1" (shape input) (at 152.4 84.455 0) (fields_autoplaced)
     (effects (font (size 1.27 1.27)) (justify left))
-    (property "Intersheetrefs" "${INTERSHEET_REFS}" (at 159.781 84.455 0)
+    (property "Intersheetrefs" "${INTERSHEET_REFS}" (at 157.3015 84.455 0)
       (effects (font (size 1.27 1.27)) (justify left) hide)
     )
@@
     )
   )
-  (global_label "col2" (shape input) (at 152.4 104.775 0) (fields_autoplaced)
+  (global_label "c2" (shape input) (at 152.4 104.775 0) (fields_autoplaced)
     (effects (font (size 1.27 1.27)) (justify left))
-    (property "Intersheetrefs" "${INTERSHEET_REFS}" (at 159.4181 104.775 0)
+    (property "Intersheetrefs" "${INTERSHEET_REFS}" (at 157.6039 104.775 0)
       (effects (font (size 1.27 1.27)) (justify left) hide)
     )
   )
-  (global_label "row2" (shape input) (at 207.645 73.025 270) (fields_autoplaced)
-    (effects (font (size 1.27 1.27)) (justify right))
-    (property "Intersheetrefs" "${INTERSHEET_REFS}" (at 207.645 80.406 90)
+  (global_label "r2" (shape input) (at 207.645 73.025 270) (fields_autoplaced)
+    (effects (font (size 1.27 1.27)) (justify right))
+    (property "Intersheetrefs" "${INTERSHEET_REFS}" (at 207.645 77.9265 90)
       (effects (font (size 1.27 1.27)) (justify right) hide)
     )
@@
     )
   )
-  (global_label "col1" (shape input) (at 152.4 89.535 0) (fields_autoplaced)
+  (global_label "c1" (shape input) (at 152.4 89.535 0) (fields_autoplaced)
     (effects (font (size 1.27 1.27)) (justify left))
-    (property "Intersheetrefs" "${INTERSHEET_REFS}" (at 159.4181 89.535 0)
+    (property "Intersheetrefs" "${INTERSHEET_REFS}" (at 157.6039 89.535 0)
       (effects (font (size 1.27 1.27)) (justify left) hide)
     )
   )
-  (global_label "row1" (shape input) (at 168.91 73.025 270) (fields_autoplaced)
-    (effects (font (size 1.27 1.27)) (justify right))
-    (property "Intersheetrefs" "${INTERSHEET_REFS}" (at 168.91 80.406 90)
+  (global_label "r1" (shape input) (at 168.91 73.025 270) (fields_autoplaced)
+    (effects (font (size 1.27 1.27)) (justify right))
+    (property "Intersheetrefs" "${INTERSHEET_REFS}" (at 168.91 77.9265 90)
       (effects (font (size 1.27 1.27)) (justify right) hide)
     )
@@
     )
   )
-  (global_label "col1" (shape input) (at 163.83 67.945 90) (fields_autoplaced)
+  (global_label "c1" (shape input) (at 163.83 67.945 90) (fields_autoplaced)
     (effects (font (size 1.27 1.27)) (justify left))
-    (property "Intersheetrefs" "${INTERSHEET_REFS}" (at 163.83 60.9269 90)
+    (property "Intersheetrefs" "${INTERSHEET_REFS}" (at 163.83 62.7411 90)
       (effects (font (size 1.27 1.27)) (justify left) hide)
     )
@@
     )
   )
-  (global_label "row2" (shape input) (at 152.4 99.695 0) (fields_autoplaced)
+  (global_label "r2" (shape input) (at 152.4 99.695 0) (fields_autoplaced)
     (effects (font (size 1.27 1.27)) (justify left))
-    (property "Intersheetrefs" "${INTERSHEET_REFS}" (at 159.781 99.695 0)
+    (property "Intersheetrefs" "${INTERSHEET_REFS}" (at 157.3015 99.695 0)
       (effects (font (size 1.27 1.27)) (justify left) hide)
     )
@@
     )
   )
-  (global_label "col2" (shape input) (at 202.565 67.945 90) (fields_autoplaced)
+  (global_label "c2" (shape input) (at 202.565 67.945 90) (fields_autoplaced)
     (effects (font (size 1.27 1.27)) (justify left))
-    (property "Intersheetrefs" "${INTERSHEET_REFS}" (at 202.565 60.9269 90)
+    (property "Intersheetrefs" "${INTERSHEET_REFS}" (at 202.565 62.7411 90)
       (effects (font (size 1.27 1.27)) (justify left) hide)
     )
@@
         )
       )
+    )
+  )
+  (symbol (lib_id "Regulator_Linear:XC6206PxxxMR") (at 172.72 161.925 0) (unit 1)
+    (in_bom yes) (on_board yes) (dnp no) (fields_autoplaced)
+    (property "Reference" "U8" (at 172.72 155.575 0)
+      (effects (font (size 1.27 1.27)))
+    )
+    (property "Value" "XC6206PxxxMR" (at 172.72 158.115 0)
+      (effects (font (size 1.27 1.27)))
+    )
+    (property "Footprint" "Package_TO_SOT_SMD:SOT-23-3" (at 172.72 156.21 0)
+      (effects (font (size 1.27 1.27) italic) hide)
+    )
+    (property "Datasheet" "https://www.torexsemi.com/file/xc6206/XC6206.pdf" (at 172.72 161.925 0)
+      (effects (font (size 1.27 1.27)) hide)
+    )
+    (pin "1")
+    (pin "2")
+    (pin "3")
+    (instances
+      (project "pandemonium BLE"
+        (path "/d73b7c39-1103-4a4e-9b7b-eba7e04e02d3"
+          (reference "U8") (unit 1)
+        )
+      )

Commit message: BLE version close to proto run
implement john's last suggestions
Parts:
- removed D33: BLUE, LED_SMD:LED_1206_3216Metric_ReverseMount_Hole1.8x2.4mm, symbol Device:LED_Small
- removed R1: 1K, Resistor_SMD:R_0402_1005Metric, symbol Device:R_Small
- removed U1, U5, U6: 74LVC1G08, Package_TO_SOT_SMD:SOT-353_SC-70-5, symbol 74xGxx:74LVC1G08
- removed U7: XC6220-3.3V, Package_TO_SOT_SMD:SOT-23-5, symbol TK44:AP2112K-3.3V
- added SWT2: SW_Push, PCM_marbastlib-various:SW_SKHLLCA010, symbol Switch:SW_Push
- F1: footprint Fuse:Fuse_0603_1608Metric -> Fuse:Fuse_1206_3216Metric
Connections:
- net GND: now also U8.1 (GND), SWT2.2
- net nRF_VDD: now also U8.2 (VO)
- net at D38.1 (K), Q1.2 (S): now also U8.3 (VI)
- net BLUE_LED renamed WakeUp
- net WakeUp: now also SWT2.1
- net WAKESLEEP renamed P0.10
Other:
- note added: "Charger and red LED for battery indicator"
- note added: "Wake up Button"
- note removed: "CHANGE LDO, ADD SIMPLE PUSH BUTTON FOR solution, needs GPIO EVQP4HB3B"
- note removed: "Charger and blue LED"
- note removed: "hardware/software wakeup"
- moved on the sheet: D38, D39, J7, Q1, R2, R3, R4, R5, R6, U3, U8
