File: Project/pandemonium.kicad_sch (KiCad schematic)
At the start: 88 parts, among them J1 XIAO nrf52840, J2 Conn_01x02_Female, J3 Conn_01x03_Female

Commit message: fresh gerbers, easier THT labelling
Parts:
- D1, D10, D11, D12, D13, D14, D15, D16, D17, D18, D19, D2, D20, D21, D22, D23, D24, D25, D26, D27, D28, D29, D3, D31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: footprint Keebio-Parts:Diode-Hybrid-Back -> kbd:D3_TH_SMD_v2
