File: Project/EC variant/pandemonium EC 2 Layer.kicad_pcb (KiCad board)
At the start: 2 copper layers, 190.5 x 81.6 mm, 105 parts, among them J1 USB_C_Receptacle_USB2.0, SW1 DFU, U11 PRTR5V0U2X, U5 OPA354, U6 74HC4051, U7 74HC4051, U8 STM32F072CBT6, U9 XC6206PxxxMR-Regulator_Linear

Commit message: backup
Routing:
- net AMUX_SEL_0: track 160.5 -> 159.0 mm
Changed lines of the file:
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@@
     (effects (font (size 1 1) (thickness 0.15)) (justify bottom mirror))
+  )
+  (gr_text "boot" (at 50.8 48.41875) (layer "B.SilkS")
+    (effects (font (size 1 1) (thickness 0.2) bold) (justify mirror))
   )
   (gr_text "ISO" (at 219.86875 81.75625) (layer "B.SilkS")
@@
   (gr_text "concept by haizeus" (at 188.11875 101.6) (layer "F.SilkS")
     (effects (font (size 1 1) (thickness 0.2) bold) (justify left bottom))
-  )
-  (gr_text "boot" (at 50.8 48.41875) (layer "F.SilkS")
-    (effects (font (size 1 1) (thickness 0.2) bold))
   )
   (via (at 161.925 95.25) (size 0.8) (drill 0.4) (layers "F.Cu" "B.Cu") (net 0))
@@
   (segment (start 93.443348 80.61875) (end 91.771466 82.290632) (width 0.25) (layer "B.Cu") (net 35))
   (segment (start 83.54441 85.90407) (end 84.936168 85.90407) (width 0.25) (layer "B.Cu") (net 35))
-  (segment (start 91.771466 82.290632) (end 90.70709 83.355008) (width 0.25) (layer "B.Cu") (net 35))
   (segment (start 164.50691 86.01202) (end 166.61324 86.01202) (width 0.25) (layer "B.Cu") (net 35))
   (segment (start 56.60625 85.125) (end 56.60625 87.882) (width 0.25) (layer "B.Cu") (net 35))

Commit message: changes to topre version and BLE version
Parts:
- added H21: MountingHole, cipulot_parts:HOLE_M2, F.Cu at (121.9, 88.0)
- added H22: MountingHole, cipulot_parts:HOLE_M2, F.Cu at (132.0, 88.0)
- added H23: MountingHole, cipulot_parts:HOLE_M2, F.Cu at (83.3, 95.2)
- added H24: MountingHole, cipulot_parts:HOLE_M2, F.Cu at (170.7, 95.2)
- added H25: MountingHole, cipulot_parts:HOLE_M2, F.Cu at (217.7, 97.3)
- moved H15 7.43 mm to (89.2, 88.1)
- moved H17 7.38 mm to (164.8, 88.1)
- moved H13 7.19 mm to (217.8, 64.6)
- moved R24 4.05 mm to (166.7, 84.4), turned to 90 degrees
- moved C31 3.97 mm to (77.0, 81.8)
- moved C32 3.97 mm to (166.7, 81.9)
- moved R16 3.97 mm to (77.0, 83.9)
- moved R17 3.97 mm to (83.3, 88.9)
- moved R18 3.97 mm to (81.8, 80.7)
- moved R19 3.97 mm to (77.0, 85.7)
- moved R21 3.97 mm to (87.3, 85.7)
- moved R25 3.97 mm to (172.6, 80.8)
- moved R26 3.97 mm to (171.4, 89.0)
- moved R27 3.97 mm to (170.7, 80.8)
- moved R28 3.97 mm to (177.0, 84.6)
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Routing:
- net COL5: track 81.6 -> 91.8 mm
- net AMUX_SEL_2: track 156.0 -> 162.1 mm
- net APLEX_EN_PIN_0: track 70.8 -> 66.2 mm
- net APLEX_OUT: track 128.9 -> 133.4 mm
- net COL3: track 86.9 -> 91.4 mm
- net AMUX_SEL_1: track 155.1 -> 159.2 mm
- net COL7: track 92.1 -> 96.2 mm
- net COL8: track 75.8 -> 71.8 mm
- net COL0: track 96.6 -> 92.6 mm
- net +3V3: track 271.4 -> 275.4 mm
- net APLEX_EN_PIN_1: track 153.6 -> 157.3 mm
- net COL9: track 115.9 -> 112.3 mm
- net COL4: track 98.3 -> 101.8 mm
- net AMUX_SEL_0: track 159.0 -> 162.4 mm
- net COL6: track 60.7 -> 63.9 mm
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Other:
- board text removed: "ADJUST SCREW HOLE FOR 2U"
- board text removed: "REDO ALL THE VIAS"
