File: Project/WIP variants/pandemonium BLE e7.kicad_sch (KiCad schematic)
At the start: 131 parts, among them J1 HRO_TYPE-C-31-M-14, J1 TC2030_SWD, J3 78171-0002, SW1 RotaryEncoder_Switch, SW2 RotaryEncoder_Switch, SW3 RST, U1 nRF52840_E73-2G4M08S1C, U4 USBLC6-2P6, U5 74LVC1G11, U6 MAX17048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

Commit message: integrated wip
Parts:
- removed C1: 100nF, Capacitor_SMD:C_0402_1005Metric, symbol Device:C_Small
- removed C11: 100n, Capacitor_SMD:C_0402_1005Metric, symbol Device:C_Small
- removed U4: USBLC6-2P6, Package_TO_SOT_SMD:SOT-666, symbol Power_Protection:USBLC6-2P6
- removed U5: 74LVC1G11, Package_TO_SOT_SMD:SOT-363_SC-70-6, symbol 74xGxx:74LVC1G11
- added SW4: SW_SPDT, PCM_marbastlib-various:SW_MSK12C02-HB, symbol Switch:SW_SPDT
- added U2: SRV05-4, PCM_marbastlib-various:SOT-23-6-routable, symbol PCM_marbastlib-various:SRV05-4
Connections:
- net DATA ESD+ is gone; now on net D+: J1.A6 (D+), J1.B6 (D+)
- net DATA ESD- is gone; now on net D-: J1.A7 (D-), J1.B7 (D-)
- net +5V: now also L5.2
- net +BATT: now also SW4.2 (B); no longer J3.1 (Pin_1)
- net D+: now also U2.1 (IO1)
- net D-: now also U2.6 (IO4)
- net GND: now also U2.2 (VN)
- net VBUS: now also F1.1, U2.5 (VP); no longer F1.2, L5.1
- net wk: no longer names the net of U1.22 (P0.07)
- new net: F1.2, L5.1
- new net: J3.1 (Pin_1), SW4.1 (A)
- no-connect marks 13 -> 17
Other:
- note removed: "AND gate for ZMK soft poweroff feature"
- note removed: "MCU e73"
- note removed: "VBUS 5+V CHECK"
- moved on the sheet: C10, C12, C13, C14, C15, C16, C17, C18, C19, C6, C7, C8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
