File: Project/WIP variants/pandemonium BLE e7 cutout.kicad_pcb (KiCad board)
At the start: 2 copper layers, 188.9 x 79.7 mm, 137 parts, among them J1 TC2030_SWD, J2 HRO_TYPE-C-31-M-14, J3 78171-0002, J4 Conn_01x02_Female, Q1 2N7002, SW1 RotaryEncoder_Switch, SW2 RotaryEncoder_Switch, SW3 RST, SW4 SW_SPDT, U1 nRF52840_E73-2G4M08S1C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

Commit message: BLE & EC edited
requires production files!!
Parts:
- removed J2: HRO_TYPE-C-31-M-14, PCM_marbastlib-various:USB_C_Receptacle_HRO_TYPE-C-31-M-12
- removed R7, R9: 5.1k, Resistor_SMD:R_0402_1005Metric
- removed U2: SRV05-4, PCM_marbastlib-various:SOT-23-6-routable
- added G***: LOGO, LOGO, F.Cu at (36.5, 97.6)
- added G***: LOGO, LOGO, B.Cu at (218.3, 102.4)
- added G***: LOGO, LOGO, B.Cu at (218.3, 98.4)
- added J5: SM04B, Connector_JST:JST_SH_SM04B-SRSS-TB_1x04-1MP_P1.00mm_Horizontal, B.Cu at (165.1, 41.3)
- moved G*** 181.8 mm to (36.5, 101.6)
- moved C12 49.8 mm to (174.8, 42.9)
- moved L2 49.8 mm to (173.8, 42.9)
- moved F2 48.6 mm to (170.7, 42.9), turned to 0 degrees
Routing:
- net D-: track 92.7 -> 44.8 mm
- net D+: track 91.7 -> 45.5 mm
- net GND: track 603.8 -> 585.8 mm, vias 32 -> 30
- net /CC1: track 10.9 -> 0.00 mm
- net VBUS: track 12.8 -> 2.19 mm, vias 2 -> 0
- net /CC2: track 9.52 -> 0.00 mm
- net +5V: track 109.9 -> 119.1 mm
- net VDD: track 195.3 -> 202.3 mm
- net +VSW: track 79.8 -> 86.2 mm
- net ROW0: track 181.8 -> 178.6 mm
- net LED_G: track 186.3 -> 184.0 mm
- net LED_B: track 185.4 -> 184.2 mm
- net SDA: track 84.0 -> 83.3 mm
Other:
- board size 188.9 x 79.7 mm -> 188.9 x 80.8 mm
- board text added: "db"
