File: Project/WIP variants/pandemonium BLE e7 cutout.kicad_sch (KiCad schematic)
At the start: 130 parts, among them J1 HRO_TYPE-C-31-M-14, J1 TC2030_SWD, J3 78171-0002, J4 Conn_01x02_Female, SW1 RotaryEncoder_Switch, SW2 RotaryEncoder_Switch, SW3 RST, SW4 SW_SPDT, U1 nRF52840_E73-2G4M08S1C, U2 SRV05-4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

Commit message: battery charging sysoff added
Parts:
- added Q1: 2N7002, Package_TO_SOT_SMD:SOT-23, symbol Transistor_FET:2N7002
- added R2: 10k, Resistor_SMD:R_0402_1005Metric, symbol Device:R_Small
- added R3: 100R, Resistor_SMD:R_0402_1005Metric, symbol Device:R_Small
- added R4: 100K, Resistor_SMD:R_0402_1005Metric, symbol Device:R_Small
Connections:
- net +5V: now also R3.1
- net +BATT: now also J3.1 (Pin_1), J4.1 (Pin_1), R4.1; no longer SW4.2 (B)
- net GND: now also J3.MP (MountPin), SW4.3 (C), Q1.2 (S), R2.2; no longer U7.15 (SYSOFF)
- removed net BATSWITCH: J3.1 (Pin_1), J4.1 (Pin_1), SW4.1 (A)
- new net: Q1.1 (G), R2.1, R3.2
- new net: R4.2, SW4.1 (A)
- new net SYSOFF: Q1.3 (D), SW4.2 (B), U7.15 (SYSOFF)
- no-connect marks 17 -> 15
Other:
- note added: "Battery connectors + on/off switch"
- note added: "Connector"
- note removed: "Battery connectors"
- moved on the sheet: J3, J4, SW4

Commit message: BLE & EC edited
requires production files!!
Parts:
- removed J1: HRO_TYPE-C-31-M-14, PCM_marbastlib-various:USB_C_Receptacle_HRO_TYPE-C-31-M-12, symbol Connector:USB_C_Receptacle_USB2.0
- removed R4, R5: 5.1k, Resistor_SMD:R_0402_1005Metric, symbol Device:R_Small
- removed U2: SRV05-4, PCM_marbastlib-various:SOT-23-6-routable, symbol PCM_marbastlib-various:SRV05-4
- added J5: SM04B, Connector_JST:JST_SH_SM04B-SRSS-TB_1x04-1MP_P1.00mm_Horizontal, symbol Connector:Conn_01x04_Female
Connections:
- net D+: now also J5.3 (Pin_3)
- net D-: now also J5.2 (Pin_2)
- net GND: now also J5.4 (Pin_4)
- net VBUS: now also J5.1 (Pin_1)
- no-connect marks 15 -> 11
Other:
- note added: "JST DB & FUZE"
- note removed: "USB and ESD"
- moved on the sheet: F1, L5
