File: Project/WIP variants/EC variant/mounting holes.kicad_sch (KiCad schematic)
At the start: 25 parts

Commit message: EC 2 layer production files
Parts:
- removed H13, H19, H20 (x2): MountingHole, cipulot_parts:HOLE_M2, symbol Mechanical:MountingHole
- H1, H10, H11, H12, H14, H15, H16, H17, H18, H19, H2, H20, H3, H4, H5, H6, H7, H8, H9: footprint cipulot_parts:HOLE_M2 -> cipulot_parts:HOLE_M2 (no arrow)
